Commit message: add save scans save GNSS origin change the robot urdf

File: launch/include/config/robot.urdf.xacro (robot description, xacro)
@@ -25,5 +25,5 @@
     <parent link="chassis_link" />
     <child link="navsat_link" />
-    <origin xyz="0 0 0" rpy="0 0 0" />
+    <origin xyz="0.111712 -0.0457508 0.222362" rpy="0 0 0" />
   </joint>
 </robot>
